File: scd30_esp.kicad_sch (KiCad schematic)
At the start: 17 parts, among them J1 SCD30, J2 USB_C_Receptacle_USB2.0, Q3 BSS138PS, U1 TLV62569DDC, U2 ESP32-WROOM-32D, U3 CH340C

Commit message: Saved schematic
Parts:
- Q3: footprint (none) -> Package_TO_SOT_SMD:SOT-363_SC-70-6
Changed lines of the file:
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@@
 			)
 		)
-		(property "Footprint" ""
+		(property "Footprint" "Package_TO_SOT_SMD:SOT-363_SC-70-6"
 			(at 125.73 78.74 0)
 			(effects
@@
 			)
 		)
-		(property "Footprint" ""
+		(property "Footprint" "Package_TO_SOT_SMD:SOT-363_SC-70-6"
 			(at 125.73 60.96 0)
 			(effects
