File: scd30_esp.kicad_sch (KiCad schematic)
At the start: 17 parts, among them J1 SCD30, J2 USB_C_Receptacle_USB2.0, Q3 BSS138PS, U1 TLV62569DDC, U2 ESP32-WROOM-32D, U3 CH340C

Commit message: Initial schematic
Parts:
- removed U2: ESP32-WROOM-32D, RF_Module:ESP32-WROOM-32D, symbol RF_Module:ESP32-WROOM-32D
- added J4: QWIIC, Connector_JST:JST_SH_SM04B-SRSS-TB_1x04-1MP_P1.00mm_Horizontal, symbol Connector_Generic:Conn_01x04
- added J5: Touch GPIO2, TestPoint:TestPoint_Pad_D1.0mm, symbol Connector_Generic:Conn_01x01
- added J6: Touch GPIO4, TestPoint:TestPoint_Pad_D1.0mm, symbol Connector_Generic:Conn_01x01
- added U2: ESP32-WROOM-E, PCM_Espressif:ESP32-WROOM-32E, symbol PCM_Espressif:ESP32-WROOM-E
- C1: value C_Small -> 120pF; LCSC (none) -> C106996
- C2: LCSC (none) -> C45783; MPN (none) -> GRM21BZ71A226KE15L
- C3: value C_Small -> 4.7uF; LCSC (none) -> C19666; MPN (none) -> GRM21BR71A475KA73L
- C4: LCSC (none) -> C1525
- C5: LCSC (none) -> C15849
- J2: LCSC (none) -> C165948
- L1: LCSC (none) -> C435392
- Q3: footprint (none) -> Package_TO_SOT_SMD:SOT-363_SC-70-6; LCSC (none) -> C193381
- R1: LCSC (none) -> C23254
- R2: LCSC (none) -> C23146
- R3: LCSC (none) -> C25804
- R4, R5: LCSC (none) -> C6119849
- U1: value TLV62569DDC -> TPS62A02PDDCR; LCSC (none) -> C22445521
- U3: LCSC (none) -> C7464026
Connections:
- net +3V3: now also J4.2 (Pin_2), U2.2 (3V3)
- net ESP_EN: now also U2.3 (EN/CHIP_PU)
- net ESP_IO0: now also U2.25 (GPIO0/BOOT/ADC2_CH1)
- net GND: now also J4.1 (Pin_1), U2.1 (GND), U2.15 (GND), U2.38 (GND), U2.39 (GND_THERMAL)
- net MCU_RX: now also U2.34 (U0RXD/GPIO3)
- net MCU_TX: now also U2.35 (U0TXD/GPIO1)
- net SCL: now also U2.36 (GPIO22)
- net SDA: now also U2.33 (GPIO21)
- new net DISP_BUSY: U2.12 (ADC2_CH7/GPIO27)
- new net PICO: U2.37 (GPIO23)
- new net POCI: U2.31 (GPIO19)
- new net QWIIC_SCL: J4.4 (Pin_4), U2.11 (DAC_2/ADC2_CH9/GPIO26)
- new net QWIIC_SDA: J4.3 (Pin_3), U2.10 (DAC_1/ADC2_CH8/GPIO25)
- new net SCLK: U2.30 (GPIO18)
- new net TOUCH2: J5.1 (Pin_1), U2.24 (ADC2_CH2/GPIO2)
- new net TOUCH4: J6.1 (Pin_1), U2.26 (ADC2_CH0/GPIO4)
- new net ~{DISP_CS}: U2.29 (GPIO5)
- new net ~{DISP_D/C}: U2.28 (GPIO17)
- new net ~{DISP_RST}: U2.27 (GPIO16)
- no-connect marks 7 -> 9
Other:
- added sheet Waveshare E-ink (waveshare_eink.kicad_sch)
- note added: "Connectivity"
- note added: "MCU"
- note added: "Sensors"
- note added: "UI"
- note removed: "MCU and Sensor"
- moved on the sheet: C1, J1
