File: scd30_esp.kicad_pcb (KiCad board)
At the start: 2 copper layers, 24.9 x 35.8 mm, 20 parts, among them J1 SCD30, J2 USB_C_Receptacle_USB2.0, Q3 BSS138PS, U1 TLV62569DDC, U2 ESP32-WROOM-32D, U3 CH340C

Commit message: Initial schematic
Parts:
- removed the G*** at (78.1, 44.1)
- added C10: 1uF, Capacitor_SMD:C_0603_1608Metric, B.Cu at (173.9, 135.8)
- added C11: 1uF, Capacitor_SMD:C_0603_1608Metric, B.Cu at (173.9, 137.3)
- added C12: 1uF, Capacitor_SMD:C_0603_1608Metric, B.Cu at (173.9, 138.8)
- added C13: 1uF, Capacitor_SMD:C_0603_1608Metric, B.Cu at (173.9, 140.3)
- added C14: 1uF, Capacitor_SMD:C_0603_1608Metric, B.Cu at (173.9, 141.8)
- added C15: 1uF, Capacitor_SMD:C_0603_1608Metric, B.Cu at (173.9, 143.3)
- added C16: 1uF, Capacitor_SMD:C_0603_1608Metric, B.Cu at (173.9, 144.8)
- added C17: 1uF, Capacitor_SMD:C_0603_1608Metric, B.Cu at (173.9, 146.3)
- added C18: 1uF, Capacitor_SMD:C_0603_1608Metric, B.Cu at (173.9, 147.8)
- added C20: 0.1uF, Capacitor_SMD:C_0402_1005Metric, B.Cu at (171.3, 140.9)
- added C8: 4u7, Capacitor_SMD:C_0805_2012Metric, F.Cu at (131.6, 131.7)
- added C9: 4u7, Capacitor_SMD:C_0805_2012Metric, F.Cu at (131.6, 134.7)
- added D1: NSR0530HT1G, Diode_SMD:D_SOD-323, F.Cu at (126.5, 131.9)
- added D2: NSR0530HT1G, Diode_SMD:D_SOD-323, F.Cu at (126.5, 135.2)
- added D3: NSR0530HT1G, Diode_SMD:D_SOD-323, F.Cu at (126.5, 138.6)
- added D4: NSR0530HT1G, Diode_SMD:D_SOD-323, F.Cu at (126.2, 147.2)
- added J3: 24P P0.5mm waveshare E-paper display, Connector_FFC-FPC:Molex_502244-2430_1x24-1MP_P0.5mm_Horizontal, F.Cu at (172.9, 142.7)
- added J4: QWIIC, Connector_JST:JST_SH_SM04B-SRSS-TB_1x04-1MP_P1.00mm_Horizontal, F.Cu at (140.2, 125.0)
- added J5: Touch GPIO2, TestPoint:TestPoint_Pad_D1.0mm, F.Cu at (146.2, 122.7)
- added J6: Touch GPIO4, TestPoint:TestPoint_Pad_D1.0mm, F.Cu at (146.2, 125.7)
- added L2: 68uF, Inductor_SMD:L_1210_3225Metric, F.Cu at (126.4, 142.4)
- added Q1: Si1308EDL, Package_TO_SOT_SMD:SOT-323_SC-70, F.Cu at (131.4, 142.3)
- added R6: 0R47, Resistor_SMD:R_0603_1608Metric, F.Cu at (121.6, 139.0)
- added R7: 10k, Resistor_SMD:R_0603_1608Metric, F.Cu at (121.6, 141.5)
- C1: value C_Small -> 120pF
- C3: value C_Small -> 4.7uF
- U1: value TLV62569DDC -> TPS62A02PDDCR
- U2: value ESP32-WROOM-32D -> ESP32-WROOM-E; footprint RF_Module:ESP32-WROOM-32D -> PCM_Espressif:ESP32-WROOM-32E
- moved R3 67.7 mm to (93.1, 120.0), turned to 180 degrees
- moved R2 66.1 mm to (96.1, 120.0), turned to 180 degrees
- moved C3 64.2 mm to (93.6, 117.5), turned to -90 degrees
- moved U1 62.3 mm to (97.0, 117.5), turned to 180 degrees
- moved R1 61.0 mm to (101.4, 118.0), turned to -90 degrees
- moved C1 60.7 mm to (100.2, 117.5), turned to -90 degrees
- moved C2 58.5 mm to (103.2, 116.6), turned to -90 degrees
- moved L1 56.9 mm to (99.3, 114.3), turned to 0 degrees
- moved J1 50.2 mm to (129.9, 64.4)
- moved U2 42.2 mm to (97.2, 92.5), turned to 90 degrees
- moved G*** 11.8 mm to (89.1, 50.0), turned to 90 degrees
- moved Q3 1.40 mm to (76.0, 48.4)
Connections:
- U2 pad 10: unconnected-(U2-IO25-Pad10) -> /QWIIC_SDA
- U2 pad 11: unconnected-(U2-IO26-Pad11) -> /QWIIC_SCL
- U2 pad 12: unconnected-(U2-IO27-Pad12) -> /DISP_BUSY
- U2 pad 17: unconnected-(U2-SHD/SD2-Pad17) -> (no net)
- U2 pad 18: unconnected-(U2-SWP/SD3-Pad18) -> (no net)
- U2 pad 19: unconnected-(U2-SCS/CMD-Pad19) -> (no net)
- U2 pad 20: unconnected-(U2-SCK/CLK-Pad20) -> (no net)
- U2 pad 21: unconnected-(U2-SDO/SD0-Pad21) -> (no net)
- U2 pad 22: unconnected-(U2-SDI/SD1-Pad22) -> (no net)
- U2 pad 24: unconnected-(U2-IO2-Pad24) -> /TOUCH2
- U2 pad 26: unconnected-(U2-IO4-Pad26) -> /TOUCH4
- U2 pad 27: unconnected-(U2-IO16-Pad27) -> /~{DISP_RST}
- U2 pad 28: unconnected-(U2-IO17-Pad28) -> /~{DISP_D/C}
- U2 pad 29: unconnected-(U2-IO5-Pad29) -> /~{DISP_CS}
- U2 pad 30: unconnected-(U2-IO18-Pad30) -> /SCLK
- U2 pad 31: unconnected-(U2-IO19-Pad31) -> /POCI
- U2 pad 32: unconnected-(U2-NC-Pad32) -> (no net)
- U2 pad 37: unconnected-(U2-IO23-Pad37) -> /PICO
Routing:
- net +3V3: track 60.2 -> 21.4 mm, vias 5 -> 1
- net GND: track 62.7 -> 101.3 mm, vias 54 -> 8
- net /MCU_TX: track 27.4 -> 4.64 mm, vias 2 -> 1
- net /MCU_RX: track 25.0 -> 4.84 mm, vias 2 -> 1
- net /Waveshare E-ink/V_CORE: track 0.00 -> 7.20 mm, vias 0 -> 1
- net /Waveshare E-ink/VPP: track 0.00 -> 6.20 mm, vias 0 -> 1
- net /SCL: track 5.52 -> 0.00 mm
- net /Waveshare E-ink/VSH1: track 0.00 -> 5.38 mm, vias 0 -> 1
- net VBUS: track 36.7 -> 32.0 mm
- net /Waveshare E-ink/VGH: track 0.00 -> 4.56 mm, vias 0 -> 1
- net /SDA: track 4.24 -> 0.00 mm
- net /Waveshare E-ink/VCOM: track 0.00 -> 3.76 mm, vias 0 -> 1
- net Net-(J3-Pin_4): track 0.00 -> 3.67 mm, vias 0 -> 1
- net /Waveshare E-ink/VSL: track 0.00 -> 3.67 mm, vias 0 -> 1
- net /Waveshare E-ink/VSH2: track 0.00 -> 3.34 mm, vias 0 -> 1
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Other:
- board text added: "SCD30 ESP32 board"
- board text added: "sche.cc/scd30esp"

Commit message: Initial layout
Parts:
- removed J5: Touch GPIO2, TestPoint:TestPoint_Pad_D1.0mm
- removed J6: Touch GPIO4, TestPoint:TestPoint_Pad_D1.0mm
- added R8: 2k2, Resistor_SMD:R_0603_1608Metric, F.Cu at (120.7, 115.0)
- added R9: 2k2, Resistor_SMD:R_0603_1608Metric, F.Cu at (122.3, 115.0)
- added SW1: SW_SPST, Button_Switch_SMD:SW_SPST_Omron_B3FS-100xP, B.Cu at (146.3, 70.3)
- C10, C11, C12, C13, C14, C15, C16, C17, C18, C20, C4, J2, Q3, U2, U3: moved to F.Cu
- J3: footprint Connector_FFC-FPC:Molex_502244-2430_1x24-1MP_P0.5mm_Horizontal -> FCI fpc:AMPHENOL_SFV24R-4STE1HLF
- moved C5 90.6 mm to (148.0, 95.2), turned to 0 degrees
- moved R4 77.3 mm to (122.3, 88.0), turned to -90 degrees
- moved C4 74.0 mm to (135.4, 86.0), turned to 90 degrees
- moved J3 72.4 mm to (114.4, 99.9), turned to -90 degrees
- moved U3 72.1 mm to (129.7, 86.2), turned to -90 degrees
- moved C10 70.3 mm to (118.6, 92.3), turned to 90 degrees
- moved Q3 70.3 mm to (130.8, 92.5)
- moved R5 70.3 mm to (122.3, 82.3), turned to 90 degrees
- moved C11 70.1 mm to (120.1, 92.3), turned to 90 degrees
- moved C17 70.1 mm to (118.7, 103.1), turned to 90 degrees
- moved C16 70.0 mm to (127.6, 92.3), turned to 90 degrees
- moved C12 70.0 mm to (121.6, 92.3), turned to 90 degrees
- moved C18 69.9 mm to (120.2, 103.1), turned to 90 degrees
- moved C15 69.9 mm to (126.1, 92.3), turned to 90 degrees
- moved C13 69.9 mm to (123.1, 92.3), turned to 90 degrees
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Connections:
- C18 pad 1: Net-(J3-Pin_4) -> Net-(J3-Pin_21)
- J3 pad 1: unconnected-(J3-Pin_1-Pad1) -> /Waveshare E-ink/VCOM
- J3 pad 10: /~{DISP_RST} -> +3V3
- J3 pad 11: /~{DISP_D/C} -> /DISP_SDA
- J3 pad 12: /~{DISP_CS} -> /SCLK
- J3 pad 13: /SCLK -> /~{DISP_CS}
- J3 pad 14: /PICO -> /~{DISP_D/C}
- J3 pad 15: +3V3 -> /~{DISP_RST}
- J3 pad 16: +3V3 -> /DISP_BUSY
- J3 pad 18: /Waveshare E-ink/V_CORE -> /Waveshare E-ink/TSDA
- J3 pad 19: /Waveshare E-ink/VPP -> /Waveshare E-ink/TSCL
- J3 pad 2: /Waveshare E-ink/GDR -> /Waveshare E-ink/VGL
- J3 pad 20: /Waveshare E-ink/VSH1 -> /Waveshare E-ink/VSH2
- J3 pad 21: /Waveshare E-ink/VGH -> Net-(J3-Pin_21)
- J3 pad 22: /Waveshare E-ink/VSL -> /Waveshare E-ink/RESE
- J3 pad 23: /Waveshare E-ink/VGL -> /Waveshare E-ink/GDR
- J3 pad 24: /Waveshare E-ink/VCOM -> unconnected-(J3-Pin_24-Pad24)
- J3 pad 3: /Waveshare E-ink/RESE -> /Waveshare E-ink/VSL
- J3 pad 4: Net-(J3-Pin_4) -> /Waveshare E-ink/VGH
- J3 pad 5: /Waveshare E-ink/VSH2 -> /Waveshare E-ink/VSH1
- J3 pad 6: /Waveshare E-ink/TSCL -> /Waveshare E-ink/VPP
- J3 pad 7: /Waveshare E-ink/TSDA -> /Waveshare E-ink/V_CORE
- J3 pad 9: /DISP_BUSY -> +3V3
- U2 pad 10: /QWIIC_SDA -> unconnected-(U2-DAC_1/ADC2_CH8/GPIO25-Pad10)
- U2 pad 11: /QWIIC_SCL -> unconnected-(U2-DAC_2/ADC2_CH9/GPIO26-Pad11)
- U2 pad 23: unconnected-(U2-MTDO/GPIO15/ADC2_CH3-Pad23) -> /QWIIC_SDA
- U2 pad 24: /TOUCH2 -> /QWIIC_SCL
- U2 pad 26: /TOUCH4 -> /BTN
- U2 pad 31: /POCI -> /DISP_SDA
- U2 pad 37: /PICO -> unconnected-(U2-GPIO23-Pad37)
Routing:
- net +3V3: track 21.4 -> 124.1 mm, vias 1 -> 4
- net GND: track 101.3 -> 158.9 mm, vias 8 -> 116
- net /MCU_TX: track 4.64 -> 46.3 mm, vias 1 -> 2
- net /MCU_RX: track 4.84 -> 44.5 mm, vias 1 -> 2
- net /SCLK: track 0.00 -> 31.9 mm, vias 0 -> 2
- net /SCL: track 0.00 -> 31.2 mm
- net /DISP_SDA: track 0.00 -> 31.1 mm, vias 0 -> 2
- net /~{DISP_D/C}: track 0.00 -> 28.7 mm, vias 0 -> 2
- net /~{DISP_CS}: track 0.00 -> 27.9 mm, vias 0 -> 2
- net /~{DISP_RST}: track 0.00 -> 27.7 mm, vias 0 -> 2
- net /BTN: track 0.00 -> 22.7 mm, vias 0 -> 1
- net /SDA: track 0.00 -> 22.7 mm
- net /DISP_BUSY: track 0.00 -> 21.8 mm, vias 0 -> 2
- net /QWIIC_SDA: track 0.00 -> 19.6 mm
- net /QWIIC_SCL: track 0.00 -> 19.0 mm
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Other:
- board size 24.9 x 35.8 mm -> 38.3 x 42.9 mm
