File: pcb/waveshare_eink.kicad_sch (KiCad schematic)
At the start: 21 parts, among them J3 24P P0.5mm waveshare E-paper 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, Q1 Si1308EDL

Commit message: RC1
Parts:
- D1, D2, D3, D4: LCSC (none) -> C556393
- J3: LCSC (none) -> C5343283
Changed lines of the file:
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@@
+			)
+		)
+		(property "LCSC" "C556393"
+			(at 120.65 65.7226 0)
+			(effects
+				(font
+					(size 1.27 1.27)
+				)
+				(hide yes)
 			)
 		)
@@
 			)
 		)
+		(property "LCSC" "C556393"
+			(at 114.3 84.582 0)
+			(effects
+				(font
+					(size 1.27 1.27)
+				)
+				(hide yes)
+			)
+		)
 		(pin "1"
 		)
@@
 			)
 		)
+		(property "LCSC" "C5343283"
+			(at 201.93 116.84 0)
+			(effects
+				(font
+					(size 1.27 1.27)
+				)
+				(hide yes)
+			)
+		)
 		(pin "1"
 		)
@@
 			)
 		)
+		(property "LCSC" "C556393"
+			(at 86.36 63.8174 0)
+			(effects
+				(font
+					(size 1.27 1.27)
+				)
+				(hide yes)
+			)
+		)
 		(pin "1"
 		)
@@
 			(effects
 				(font
+					(size 1.27 1.27)
+				)
+				(hide yes)
+			)
+		)
+		(property "LCSC" "C556393"
+			(at 127.254 84.836 0)
+			(effects
+				(font

Commit message: Added JLCPCB production files
Parts:
- L2: LCSC (none) -> C223228
- Q1: LCSC (none) -> C469327
Changed lines of the file:
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@@
+			)
+		)
+		(property "LCSC" "C223228"
+			(at 93.98 66.04 0)
+			(effects
+				(font
+					(size 1.27 1.27)
+				)
+				(hide yes)
 			)
 		)
@@
 			(effects
 				(font
+					(size 1.27 1.27)
+				)
+				(hide yes)
+			)
+		)
+		(property "LCSC" "C469327"
+			(at 106.934 77.47 0)
+			(effects
+				(font
